Commit message: Add 2019 FRC field description for gazebo Update ros_control_boilerplate to better match the plans for gazebosim -  mainly move all init code out of the constructors and into init() Create and hook up a frcrobot_gazebosim plugin. It loads but crashes

File: zebROS_ws/src/frcrobot_description/frcrobot_description/urdf/frcrobot.xacro (robot description, xacro)
@@ -20,5 +20,5 @@
 			</visual>
 			<collision>
-				<origin xyz="0 0 -${swerve_box_size / 2}" rpy="0 0 0"/>
+				<origin xyz="0 0 ${swerve_box_size / 2}" rpy="0 0 0"/>
 				<geometry>
 					<box size="${swerve_box_size} ${swerve_box_size} ${swerve_box_size}"/>
@@ -27,4 +27,5 @@
 			<inertial>
 				<mass value="0.5"/>
+				<origin xyz="0 0 ${swerve_box_size/2}" rpy="0 0 0"/>
 				<inertia ixx="0.1" iyy="0.1" izz="0.1" ixy="0.0" ixz="0.0" iyz="0.0"/>
 			</inertial>
@@ -79,5 +80,6 @@
 		</collision>
 		<inertial>
-		  <mass value="10.0"/>
+		  <mass value="50.0"/>
+		  <origin xyz="0 0 ${-base_height}" rpy="0 0 0"/>
 		  <inertia ixx="1.0" iyy="1.0" izz="1.0" ixy="0.0" ixz="0.0" iyz="0.0"/>
 		</inertial>
@@ -99,4 +101,13 @@
 			</material>
 		</visual>
+		<collision>
+			<geometry>
+				<box size="${elevator_width} 0.05 ${elevator_height}"/>
+			</geometry>
+		</collision>
+		<inertial>
+		  <mass value="10.0"/>
+		  <inertia ixx="1.0" iyy="1.0" izz="1.0" ixy="0.0" ixz="0.0" iyz="0.0"/>
+		</inertial>
 	</link>
 	<joint name="elevator_plate_to_base_link" type="fixed">
@@ -105,4 +116,10 @@
 		<origin xyz="-0.25 0 ${elevator_height/2 + base_height/2}" rpy="0 0 ${pi/2}"/>
 	</joint>
+	<gazebo>
+		<plugin name="gazebo_ros_plugin" filename="libgazebo_ros_control.so">
+			<robotNamespace>/frcrobot</robotNamespace>
+			<robotSimType>frcrobot_control/FRCRobotGazeboSim</robotSimType>
+		</plugin>
+	</gazebo>
 	<xacro:swerve_module prefix="lf" x="${base_width/2 - swerve_box_size/2}" y="${base_depth/2 - swerve_box_size/2}"/>
 	<xacro:swerve_module prefix="rf" x="${base_width/2 - swerve_box_size/2}" y="-${base_depth/2 - swerve_box_size/2}"/>

Commit message: Gazebosim fixes (still not working tho)

File: zebROS_ws/src/frcrobot_description/frcrobot_description/urdf/frcrobot.xacro (robot description, xacro)
@@ -52,5 +52,5 @@
 			</inertial>
 		</link>
-		<joint name="base_to_${prefix}_angle" type="continuous">
+		<joint name="${prefix}_angle" type="continuous">
 			<parent link="base_plate"/>
 			<child link="${prefix}_angle"/>
@@ -58,5 +58,5 @@
 			<axis xyz="0 0 1" />
 		</joint>
-		<joint name="${prefix}_angle_to_speed" type="continuous">
+		<joint name="${prefix}_drive" type="continuous">
 			<parent link="${prefix}_angle"/>
 			<child link="${prefix}_speed"/>
@@ -118,12 +118,12 @@
 	<gazebo>
 		<plugin name="gazebo_ros_plugin" filename="libgazebo_ros_control.so">
-			<robotNamespace>/frcrobot</robotNamespace>
+			<robotNamespace>/frcrobot_jetson</robotNamespace>
 			<robotSimType>frcrobot_control/FRCRobotGazeboSim</robotSimType>
 		</plugin>
 	</gazebo>
-	<xacro:swerve_module prefix="lf" x="${base_width/2 - swerve_box_size/2}" y="${base_depth/2 - swerve_box_size/2}"/>
-	<xacro:swerve_module prefix="rf" x="${base_width/2 - swerve_box_size/2}" y="-${base_depth/2 - swerve_box_size/2}"/>
-	<xacro:swerve_module prefix="lr" x="-${base_width/2 - swerve_box_size/2}" y="${base_depth/2 - swerve_box_size/2}"/>
-	<xacro:swerve_module prefix="rr" x="-${base_width/2 - swerve_box_size/2}" y="-${base_depth/2 - swerve_box_size/2}"/>
+	<xacro:swerve_module prefix="fl" x="${base_width/2 - swerve_box_size/2}" y="${base_depth/2 - swerve_box_size/2}"/>
+	<xacro:swerve_module prefix="fr" x="${base_width/2 - swerve_box_size/2}" y="-${base_depth/2 - swerve_box_size/2}"/>
+	<xacro:swerve_module prefix="bl" x="-${base_width/2 - swerve_box_size/2}" y="${base_depth/2 - swerve_box_size/2}"/>
+	<xacro:swerve_module prefix="br" x="-${base_width/2 - swerve_box_size/2}" y="-${base_depth/2 - swerve_box_size/2}"/>
 	<xacro:include filename="$(find controller_node)/urdf/2019_compbot.urdf"/>
 </robot>

Commit message: Robot kinda drives in gazebo - need to fix motion magic profiles

File: zebROS_ws/src/frcrobot_description/frcrobot_description/urdf/frcrobot.xacro (robot description, xacro)
@@ -20,5 +20,7 @@
 			</visual>
 			<collision>
+				<!--
 				<origin xyz="0 0 ${swerve_box_size / 2}" rpy="0 0 0"/>
+-->
 				<geometry>
 					<box size="${swerve_box_size} ${swerve_box_size} ${swerve_box_size}"/>
@@ -61,5 +63,5 @@
 			<parent link="${prefix}_angle"/>
 			<child link="${prefix}_speed"/>
-			<origin xyz="0 0 -${wheel_diameter}" rpy="0 0 0"/>
+			<origin xyz="0 0 -${wheel_diameter+.001}" rpy="0 0 0"/>
 			<axis xyz="0 1 0" />
 		</joint>

Commit message: Minor updates to gazebosim specs

File: zebROS_ws/src/frcrobot_description/frcrobot_description/urdf/frcrobot.xacro (robot description, xacro)
@@ -28,5 +28,5 @@
 			</collision>
 			<inertial>
-				<mass value="0.5"/>
+				<mass value="0.1"/>
 				<origin xyz="0 0 ${swerve_box_size/2}" rpy="0 0 0"/>
 				<inertia ixx="0.1" iyy="0.1" izz="0.1" ixy="0.0" ixz="0.0" iyz="0.0"/>
@@ -50,5 +50,5 @@
 			</collision>
 			<inertial>
-				<mass value="0.5"/>
+				<mass value="0.1"/>
 				<inertia ixx="0.1" iyy="0.1" izz="0.1" ixy="0.0" ixz="0.0" iyz="0.0"/>
 			</inertial>
@@ -82,5 +82,5 @@
 		</collision>
 		<inertial>
-		  <mass value="50.0"/>
+		  <mass value="55.0"/>
 		  <origin xyz="0 0 ${-base_height}" rpy="0 0 0"/>
 		  <inertia ixx="1.0" iyy="1.0" izz="1.0" ixy="0.0" ixz="0.0" iyz="0.0"/>

Commit message: Add solenoid control to gazebosim

File: zebROS_ws/src/frcrobot_description/frcrobot_description/urdf/frcrobot.xacro (robot description, xacro)
@@ -118,4 +118,26 @@
 		<origin xyz="-0.25 0 ${elevator_height/2 + base_height/2}" rpy="0 0 ${pi/2}"/>
 	</joint>
+	<link name="hatch_grabber_arm">
+		<visual>
+			<geometry>
+				<box size=".3 .05 .05"/>
+			</geometry>
+		</visual>
+		<collision>
+			<geometry>
+				<box size=".3 .05 .05"/>
+			</geometry>
+		</collision>
+		<inertial>
+		  <mass value="2.0"/>
+		  <inertia ixx="1.0" iyy="1.0" izz="1.0" ixy="0.0" ixz="0.0" iyz="0.0"/>
+		</inertial>
+	</link>
+	<joint name="panel_push_extend" type="prismatic">
+		<parent link="elevator_plate"/>
+		<child link="hatch_grabber_arm"/>
+		<origin xyz="-0.1 -0.05 ${-elevator_height/3.5}" rpy="${-pi/2} ${pi} 0"/>
+		<limit effort="30" velocity="1.0" lower="0.0" upper="0.3" />
+	</joint>
 	<!--
 	<gazebo>
